File: Shoto.kicad_pcb (KiCad board)
At the start: 2 copper layers, 99 parts, among them K1 KEYSW, K10 KEYSW, K11 KEYSW, K12 KEYSW, K13 KEYSW, K14 KEYSW, K15 KEYSW, K16 KEYSW, K17 KEYSW, K18 KEYSW, K19 KEYSW, K2 KEYSW, K20 KEYSW, K21 KEYSW, K22 KEYSW, K23 KEYSW, K24 KEYSW, K25 KEYSW, K26 KEYSW, K27 KEYSW, K28 KEYSW, K29 KEYSW, K3 KEYSW, K30 KEYSW, K31 KEYSW, K32 KEYSW, K33 KEYSW, K34 KEYSW, K35 KEYSW, K36 KEYSW, K37 KEYSW, K38 KEYSW, K39 KEYSW, K4 KEYSW, K40 KEYSW, K41 KEYSW, K42 KEYSW, K43 KEYSW, K44 KEYSW, K45 KEYSW, K46 KEYSW, K47 KEYSW, K48 KEYSW, K5 KEYSW, K6 KEYSW, K7 KEYSW, K8 KEYSW, K9 KEYSW, U1 STM32F030C6Tx

Commit message: ready for production
Parts:
- removed D1, D10, D11, D12, D13, D14, D15, D16, D17, D18, D19, D2, D20, D21, D22, D23, D24, D25, D26, D27, D28, D29, D3, D30, D31, D32, D33, D34, D35, D36, D37, D38, D39, D4, D40, D41, D42, D43, D44, D45, D46, D47, D48, D5, D6, D7, D8, D9: D, Diode_SMD:D_0805_2012Metric_Pad1.15x1.40mm_HandSolder
- removed REF** (x2): 2U, Keebio-Parts:2U-StabFlip
- removed U1: STM32F030C6Tx, Package_QFP:LQFP-48_7x7mm_P0.5mm
- added C101: 100n, Capacitor_SMD:C_0603_1608Metric, B.Cu at (168.5, 95.2)
- added C102: 100n, Capacitor_SMD:C_0603_1608Metric, B.Cu at (150.8, 95.3)
- added C103: 100n, Capacitor_SMD:C_0603_1608Metric, B.Cu at (158.0, 86.1)
- added C104: 10n, Capacitor_SMD:C_0603_1608Metric, B.Cu at (161.8, 102.8)
- added C105: 4.7u, Capacitor_SMD:C_0603_1608Metric, B.Cu at (166.5, 95.2)
- added C106: 4.7u, Capacitor_SMD:C_0603_1608Metric, B.Cu at (158.0, 87.8)
- added C107: 1u, Capacitor_SMD:C_0603_1608Metric, B.Cu at (158.2, 102.8)
- added C108: 4.7u, Capacitor_SMD:C_0603_1608Metric, B.Cu at (149.0, 95.3)
- added C109: 4.7n, Capacitor_SMD:C_0603_1608Metric, B.Cu at (69.2, 31.8)
- added C110: 1u, Capacitor_SMD:C_0603_1608Metric, B.Cu at (148.1, 53.1)
- added C111: 1u, Capacitor_SMD:C_0603_1608Metric, B.Cu at (154.6, 52.8)
- added C112: 10u, Capacitor_SMD:C_0603_1608Metric, B.Cu at (182.2, 48.2)
- added C113: 1u, Capacitor_SMD:C_0603_1608Metric, B.Cu at (183.0, 51.2)
- added D101: SMF9.0CA, Diode_SMD:D_SOD-123, B.Cu at (86.7, 32.7)
- added D102: D_Schottky, Diode_SMD:D_SOD-123, B.Cu at (151.8, 49.0)
- added D201: D, Diode_SMD:D_SOD-123, B.Cu at (152.0, 44.8)
- added D208: D, Diode_SMD:D_SOD-123, B.Cu at (151.9, 64.8)
- added D215: D, Diode_SMD:D_SOD-123, B.Cu at (142.6, 72.2)
- added D222: D, Diode_SMD:D_SOD-123, B.Cu at (180.5, 84.0)
- added D223: D, Diode_SMD:D_SOD-123, B.Cu at (51.6, 86.2)
- added D224: D, Diode_SMD:D_SOD-123, B.Cu at (75.3, 86.2)
- added D225: D, Diode_SMD:D_SOD-123, B.Cu at (99.1, 86.2)
- added D226: D, Diode_SMD:D_SOD-123, B.Cu at (141.5, 84.0)
- added D227: D, Diode_SMD:D_SOD-123, B.Cu at (199.9, 86.2)
- added D228: D, Diode_SMD:D_SOD-123, B.Cu at (217.8, 86.2)
- added D229: D, Diode_SMD:D_SOD-123, B.Cu at (241.6, 86.2)
- added D230: D, Diode_SMD:D_SOD-123, B.Cu at (265.3, 86.0)
- added DD202: BAV70, keyboard_parts:SOT23-3_HSOL, B.Cu at (57.0, 44.4)
- added DD203: BAV70, keyboard_parts:SOT23-3_HSOL, B.Cu at (95.0, 44.4)
- added DD204: BAV70, keyboard_parts:SOT23-3_HSOL, B.Cu at (133.0, 44.4)
- added DD205: BAV70, keyboard_parts:SOT23-3_HSOL, B.Cu at (190.0, 44.4)
- added DD206: BAV70, keyboard_parts:SOT23-3_HSOL, B.Cu at (228.0, 44.4)
- added DD207: BAV70, keyboard_parts:SOT23-3_HSOL, B.Cu at (266.0, 44.4)
- added DD209: BAV70, keyboard_parts:SOT23-3_HSOL, B.Cu at (52.2, 65.0)
- added DD210: BAV70, keyboard_parts:SOT23-3_HSOL, B.Cu at (90.2, 65.0)
- added DD211: BAV70, keyboard_parts:SOT23-3_HSOL, B.Cu at (128.2, 65.0)
- added DD212: BAV70, keyboard_parts:SOT23-3_HSOL, B.Cu at (194.7, 65.0)
- added DD213: BAV70, keyboard_parts:SOT23-3_HSOL, B.Cu at (232.7, 65.0)
- added DD214: BAV70, keyboard_parts:SOT23-3_HSOL, B.Cu at (270.7, 65.0)
- added DD216: BAV70, keyboard_parts:SOT23-3_HSOL, B.Cu at (47.6, 71.8)
- added DD217: BAV70, keyboard_parts:SOT23-3_HSOL, B.Cu at (85.6, 71.8)
- added DD218: BAV70, keyboard_parts:SOT23-3_HSOL, B.Cu at (123.6, 71.8)
- added DD219: BAV70, keyboard_parts:SOT23-3_HSOL, B.Cu at (199.6, 71.8)
- added DD220: BAV70, keyboard_parts:SOT23-3_HSOL, B.Cu at (237.6, 71.8)
- added DD221: BAV70, keyboard_parts:SOT23-3_HSOL, B.Cu at (275.6, 71.8)
- added F101: ASMD1206-150, Fuse:Fuse_1206_3216Metric, B.Cu at (84.0, 32.7)
- added H101: MountingHole, MountingHole:MountingHole_2.2mm_M2, F.Cu at (90.0, 49.0)
- added H102: MountingHole, MountingHole:MountingHole_2.2mm_M2, F.Cu at (90.0, 87.0)
- added H103: MountingHole, MountingHole:MountingHole_2.2mm_M2, F.Cu at (109.0, 67.0)
- added H104: MountingHole, MountingHole:MountingHole_2.2mm_M2, F.Cu at (233.0, 49.0)
- added H105: MountingHole, MountingHole:MountingHole_2.2mm_M2, F.Cu at (214.0, 67.0)
- added H106: MountingHole, MountingHole:MountingHole_2.2mm_M2, F.Cu at (233.0, 87.0)
- added J101: USB_C_Receptacle_USB2.0, Connector_USB:USB_C_Receptacle_HRO_TYPE-C-31-M-12, B.Cu at (75.9, 27.2)
- added J102: Case, MountingHole:MountingHole_2.2mm_M2_Pad, B.Cu at (57.0, 31.2)
- added Q101: 2N7002, Package_TO_SOT_SMD:SOT-23, B.Cu at (180.0, 51.2)
- added R101: 5.1k, Resistor_SMD:R_0603_1608Metric, B.Cu at (72.1, 33.4)
- added R102: 5.1k, Resistor_SMD:R_0603_1608Metric, B.Cu at (79.7, 33.4)
- added R103: 1M, Resistor_SMD:R_1206_3216Metric, B.Cu at (65.6, 31.9)
- added R104: 10k, Resistor_SMD:R_0603_1608Metric, B.Cu at (174.2, 55.5)
- added R105: 10k, Resistor_SMD:R_0603_1608Metric, B.Cu at (177.0, 51.2)
- added R106: 100k, Resistor_SMD:R_0603_1608Metric, B.Cu at (180.0, 54.2)
- added SW101: TS-1187A-B-A-B, Keebio-Parts:SW_SPST_TL3342, B.Cu at (171.5, 51.1)
- added Stab_1: Stabilizer, Keebio-Parts:2U-StabFlip, F.Cu at (135.4, 95.0)
- added Stab_2: Stabilizer, Keebio-Parts:2U-StabFlip, F.Cu at (182.9, 95.0)
- added U101: STM32F072C8Tx, Package_QFP:LQFP-48_7x7mm_P0.5mm, B.Cu at (158.7, 95.3)
- added U102: XC6206PxxxMR, Package_TO_SOT_SMD:SOT-23, B.Cu at (151.6, 52.8)
- added U103: SRV05-4, Package_TO_SOT_SMD:SOT-23-6, B.Cu at (75.9, 36.4)
- turned K244 to 180 degrees
- turned K245 to 180 degrees
- renumbered K1 to K201, K2 to K202, K3 to K203, K4 to K204, K5 to K205, K6 to K206, K7 to K207, K8 to K208, K9 to K209, K10 to K210, K11 to K211, K12 to K212, K13 to K213, K14 to K214, K15 to K215, K16 to K216, K17 to K217, K18 to K218, K19 to K219, K20 to K220, K21 to K221, K22 to K222, K23 to K223, K24 to K224, K25 to K225, K26 to K226, K27 to K227, K28 to K228, K29 to K229, K30 to K230, K31 to K231, K32 to K232, K33 to K233, K35 to K234, K36 to K235, K37 to K236, K38 to K237, K39 to K238, K40 to K239, K34 to K240, K41 to K241, K42 to K242, K43 to K243, K44 to K244, K45 to K245, K46 to K246, K47 to K247, K48 to K248
Connections:
- net Net-(K1-Pad1) renamed Col_1
- net Net-(K13-Pad1) renamed Col_13
- K202 pad 1: Net-(K15-Pad1) -> Col_2
- K203 pad 1: Net-(K16-Pad1) -> Col_3
- K204 pad 1: Net-(K17-Pad1) -> Col_4
- K205 pad 1: Net-(K18-Pad1) -> Col_5
- K206 pad 1: Net-(K19-Pad1) -> Col_6
- K207 pad 1: Net-(K34-Pad1) -> Col_7
- K208 pad 1: Net-(K21-Pad1) -> Col_8
- K209 pad 1: Net-(K22-Pad1) -> Col_9
- K210 pad 1: Net-(K10-Pad1) -> Col_10
- K211 pad 1: Net-(K11-Pad1) -> Col_11
- K212 pad 1: Net-(K12-Pad1) -> Col_12
- K215 pad 1: Net-(K15-Pad1) -> Col_2
- K216 pad 1: Net-(K16-Pad1) -> Col_3
- K217 pad 1: Net-(K17-Pad1) -> Col_4
- K218 pad 1: Net-(K18-Pad1) -> Col_5
- K219 pad 1: Net-(K19-Pad1) -> Col_6
- K220 pad 1: Net-(K20-Pad1) -> Col_7
- K221 pad 1: Net-(K21-Pad1) -> Col_8
- K222 pad 1: Net-(K22-Pad1) -> Col_9
- K223 pad 1: Net-(K10-Pad1) -> Col_10
- K224 pad 1: Net-(K11-Pad1) -> Col_11
- K225 pad 1: Net-(K12-Pad1) -> Col_12
- K228 pad 1: Net-(K15-Pad1) -> Col_2
- K229 pad 1: Net-(K16-Pad1) -> Col_3
- K230 pad 1: Net-(K17-Pad1) -> Col_4
- K231 pad 1: Net-(K18-Pad1) -> Col_5
- K232 pad 1: Net-(K19-Pad1) -> Col_6
- K233 pad 1: Net-(K20-Pad1) -> Col_7
- K234 pad 1: Net-(K21-Pad1) -> Col_8
- K235 pad 1: Net-(K22-Pad1) -> Col_9
- K236 pad 1: Net-(K10-Pad1) -> Col_10
- K237 pad 1: Net-(K11-Pad1) -> Col_11
- K238 pad 1: Net-(K12-Pad1) -> Col_12
- K240 pad 1: Net-(K34-Pad1) -> Col_7
- K241 pad 1: Net-(K17-Pad1) -> Col_2
- K242 pad 1: Net-(K18-Pad1) -> Col_3
- K243 pad 1: Net-(K19-Pad1) -> Col_4
- K244 pad 1: Net-(K20-Pad1) -> Col_6
- K245 pad 1: Net-(K34-Pad1) -> Col_8
- K246 pad 1: Net-(K21-Pad1) -> Col_10
- K247 pad 1: Net-(K22-Pad1) -> Col_11
- K248 pad 1: Net-(K10-Pad1) -> Col_12
Routing:
- net Row_1: track 0.00 -> 259.5 mm, vias 0 -> 4
- net Row_3: track 0.00 -> 250.3 mm, vias 0 -> 4
- net Row_2: track 0.00 -> 247.6 mm, vias 0 -> 4
- net Row_4: track 0.00 -> 225.5 mm, vias 0 -> 2
- net Col_13: track 0.00 -> 185.2 mm, vias 0 -> 5
- net Col_12: track 0.00 -> 178.7 mm, vias 0 -> 6
- net Col_1: track 0.00 -> 167.0 mm, vias 0 -> 4
- net Col_2: track 0.00 -> 163.1 mm, vias 0 -> 6
- net D-: track 0.00 -> 159.7 mm
- net D+: track 0.00 -> 157.8 mm
- net Col_11: track 0.00 -> 156.0 mm, vias 0 -> 7
- net Col_3: track 0.00 -> 139.9 mm, vias 0 -> 6
- net Col_10: track 0.00 -> 132.9 mm, vias 0 -> 7
- net +3V3: track 0.00 -> 122.3 mm, vias 0 -> 6
- net Col_4: track 0.00 -> 116.7 mm, vias 0 -> 6
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- added copper zone on B.Cu, net GND
- added copper zone on F.Cu, net GND
Other:
- board outline added: 265.2 x 79 mm
- net class fabi added: clearance 0.2, trace_width 0.2, via_dia 0.8, via_drill 0.4

Commit message: working and produced unit
Parts:
- removed K229: KEYSW, keyboard_parts:Kailh_MX_Socket
- removed U101: STM32F072C8Tx, Package_QFP:LQFP-48_7x7mm_P0.5mm
- added G***: LOGO, Shoto:test, B.Cu at (206.5, 121.8)
- added K29: KEYSW, keyboard_parts:Kailh_MX_Socket, F.Cu at (292.0, 130.5)
- added U1: STM32F072C8Tx, Package_QFP:LQFP-48_7x7mm_P0.5mm, F.Cu at (209.3, 149.9)
- C1: renamed from C101; moved to F.Cu
- C10: renamed from C110; moved to F.Cu
- C11: renamed from C111; moved to F.Cu
- C12: renamed from C112; moved to F.Cu
- C13: renamed from C113; moved to F.Cu
- C2: renamed from C102; moved to F.Cu
- C3: renamed from C103; moved to F.Cu
- C4: renamed from C104; moved to F.Cu
- C5: renamed from C105; moved to F.Cu
- C6: renamed from C106; moved to F.Cu
- C7: renamed from C107; moved to F.Cu
- C8: renamed from C108; moved to F.Cu
- C9: renamed from C109; moved to F.Cu
- D1: renamed from D101; moved to F.Cu
- D10: renamed from D226; moved to F.Cu
- D11: renamed from D227; moved to F.Cu
- D12: renamed from D228; moved to F.Cu
- D13: renamed from D229; moved to F.Cu
- D14: renamed from D230; moved to F.Cu
- D2: renamed from D102; moved to F.Cu
- D3: renamed from D201; moved to F.Cu
- D4: renamed from D208; moved to F.Cu
- D5: renamed from D215; moved to F.Cu
- D6: renamed from D222; moved to F.Cu
- D7: renamed from D223; moved to F.Cu
- D8: renamed from D224; moved to F.Cu
- D9: renamed from D225; moved to F.Cu
- DD1: renamed from DD202; moved to F.Cu
- DD10: renamed from DD212; moved to F.Cu
- DD11: renamed from DD213; moved to F.Cu
- DD12: renamed from DD214; moved to F.Cu
- DD13: renamed from DD216; moved to F.Cu
- DD14: renamed from DD217; moved to F.Cu
- DD15: renamed from DD218; moved to F.Cu
- DD16: renamed from DD219; moved to F.Cu
- DD17: renamed from DD220; moved to F.Cu
- DD18: renamed from DD221; moved to F.Cu
- DD2: renamed from DD203; moved to F.Cu
- DD3: renamed from DD204; moved to F.Cu
- DD4: renamed from DD205; moved to F.Cu
- DD5: renamed from DD206; moved to F.Cu
- DD6: renamed from DD207; moved to F.Cu
- DD7: renamed from DD209; moved to F.Cu
- DD8: renamed from DD210; moved to F.Cu
- DD9: renamed from DD211; moved to F.Cu
- F1: renamed from F101; moved to F.Cu
- H1: renamed from H101; moved to B.Cu
- H2: renamed from H102; moved to B.Cu
- H3: renamed from H103; moved to B.Cu
- H4: renamed from H104; moved to B.Cu
- H5: renamed from H105; moved to B.Cu
- H6: renamed from H106; moved to B.Cu
- J1: renamed from J101; moved to F.Cu
- J2: renamed from J102; moved to F.Cu
- K1: renamed from K201; moved to F.Cu
- K10: renamed from K210; moved to F.Cu
- K11: renamed from K211; moved to F.Cu
- K12: renamed from K212; moved to F.Cu
- K13: renamed from K213; moved to F.Cu
- K14: renamed from K214; moved to F.Cu
- K15: renamed from K215; moved to F.Cu
- K16: renamed from K216; moved to F.Cu
- K17: renamed from K217; moved to F.Cu
- K18: renamed from K218; moved to F.Cu
- K19: renamed from K219; moved to F.Cu
- K2: renamed from K202; moved to F.Cu
- K20: renamed from K220; moved to F.Cu
- K21: renamed from K221; moved to F.Cu
- K22: renamed from K222; moved to F.Cu
- K23: renamed from K223; moved to F.Cu
- K24: renamed from K224; moved to F.Cu
- K25: renamed from K225; moved to F.Cu
- K26: renamed from K226; moved to F.Cu
- K27: renamed from K227; moved to F.Cu
- K28: renamed from K228; moved to F.Cu
- K3: renamed from K203; moved to F.Cu
- K30: renamed from K230; moved to F.Cu
- K31: renamed from K231; moved to F.Cu
- K32: renamed from K232; moved to F.Cu
- K33: renamed from K233; moved to F.Cu
- K34: renamed from K234; moved to F.Cu
- K35: renamed from K235; moved to F.Cu
- K36: renamed from K236; moved to F.Cu
- K37: renamed from K237; moved to F.Cu
- K38: renamed from K238; moved to F.Cu
- K39: renamed from K239; moved to F.Cu
- K4: renamed from K204; moved to F.Cu
- K40: renamed from K240; moved to F.Cu
- K41: renamed from K241; moved to F.Cu
- K42: renamed from K242; moved to F.Cu
- K43: renamed from K243; moved to F.Cu
- K44: renamed from K244; moved to F.Cu
- K45: renamed from K245; moved to F.Cu
- K46: renamed from K246; moved to F.Cu
- K47: renamed from K247; moved to F.Cu
- K48: renamed from K248; moved to F.Cu
- K5: renamed from K205; moved to F.Cu
- K6: renamed from K206; moved to F.Cu
- K7: renamed from K207; moved to F.Cu
- K8: renamed from K208; moved to F.Cu
- K9: renamed from K209; moved to F.Cu
- Q1: renamed from Q101; moved to F.Cu
- R1: renamed from R101; moved to F.Cu
- R2: renamed from R102; moved to F.Cu
- R3: renamed from R103; moved to F.Cu
- R4: renamed from R104; moved to F.Cu
- R5: renamed from R105; moved to F.Cu
- R6: renamed from R106; moved to F.Cu
- SW1: renamed from SW101; moved to F.Cu
- Stab_1, Stab_2: moved to B.Cu
- U2: renamed from U102; moved to F.Cu
- U3: renamed from U103; moved to F.Cu
- moved K27 297.0 mm to (330.0, 130.5), turned to 180 degrees
- moved K14 287.7 mm to (325.2, 111.5), turned to 180 degrees
- moved K1 278.4 mm to (320.5, 92.5), turned to 180 degrees
- moved DD13 278.2 mm to (320.4, 126.3), turned to 0 degrees
- moved D7 270.4 mm to (316.4, 140.7)
- moved DD7 269.2 mm to (315.8, 119.5), turned to 180 degrees
- moved K41 264.4 mm to (313.4, 149.5), turned to 180 degrees
- moved K28 259.8 mm to (311.0, 130.5), turned to 180 degrees
- moved DD1 259.8 mm to (311.0, 98.9), turned to 180 degrees
- moved J2 259.8 mm to (311.0, 85.7), turned to 180 degrees
- moved K15 250.5 mm to (306.2, 111.5), turned to 180 degrees
- moved R3 242.9 mm to (302.4, 86.4), turned to 180 degrees
- moved K2 241.2 mm to (301.5, 92.5), turned to 180 degrees
- moved C9 236.0 mm to (298.8, 86.3)
- moved R1 230.4 mm to (295.9, 87.9), turned to 180 degrees
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Routing:
- net Col_7: track 78.1 -> 79.7 mm
- net Col_9: track 112.4 -> 111.6 mm
- net +3V3: track 122.3 -> 123.0 mm
- net NRST: track 66.9 -> 67.4 mm
- net GND: track 69.9 -> 69.6 mm, vias 9 -> 12
- net (no net): vias 0 -> 1
Other:
- outline, holes or cut-outs redrawn
