File: Shoto.sch (KiCad schematic (older format))
At the start: 1 part, among them U1 STM32F030C6Tx

Commit message: ready for production
Parts:
- removed U1: STM32F030C6Tx, Package_QFP:LQFP-48_7x7mm_P0.5mm, symbol MCU_ST_STM32F0:STM32F030C6Tx
- added C101, C102, C103: 100n, Capacitor_SMD:C_0603_1608Metric, symbol Device:C
- added C104: 10n, Capacitor_SMD:C_0603_1608Metric, symbol Device:C
- added C105, C106, C108: 4.7u, Capacitor_SMD:C_0603_1608Metric, symbol Device:C
- added C107, C110, C111, C113: 1u, Capacitor_SMD:C_0603_1608Metric, symbol Device:C
- added C109: 4.7n, Capacitor_SMD:C_0603_1608Metric, symbol Device:C
- added C112: 10u, Capacitor_SMD:C_0603_1608Metric, symbol Device:C
- added D101: SMF9.0CA, Diode_SMD:D_SOD-123, symbol Diode:SD05_SOD323
- added D102: D_Schottky, Diode_SMD:D_SOD-123, symbol Device:D_Schottky
- added F101: ASMD1206-150, Fuse:Fuse_1206_3216Metric, symbol Device:Polyfuse
- added H101, H102, H103, H104, H105, H106: MountingHole, MountingHole:MountingHole_2.2mm_M2, symbol Mechanical:MountingHole
- added J101: USB_C_Receptacle_USB2.0, Connector_USB:USB_C_Receptacle_HRO_TYPE-C-31-M-12, symbol Shoto-rescue:USB_C_Receptacle_USB2.0-Connector
- added J102: Case, MountingHole:MountingHole_2.2mm_M2_Pad, symbol Connector:Conn_01x01_Female
- added Q101: 2N7002, Package_TO_SOT_SMD:SOT-23, symbol Transistor_FET:2N7002
- added R101, R102: 5.1k, Resistor_SMD:R_0603_1608Metric, symbol Device:R
- added R103: 1M, Resistor_SMD:R_1206_3216Metric, symbol Device:R
- added R104, R105: 10k, Resistor_SMD:R_0603_1608Metric, symbol Device:R
- added R106: 100k, Resistor_SMD:R_0603_1608Metric, symbol Device:R
- added SW101: TS-1187A-B-A-B, Keebio-Parts:SW_SPST_TL3342, symbol Switch:SW_Push
- added U101: STM32F072C8Tx, Package_QFP:LQFP-48_7x7mm_P0.5mm, symbol MCU_ST_STM32F0:STM32F072CBUx
- added U102: XC6206PxxxMR, Package_TO_SOT_SMD:SOT-23, symbol Regulator_Linear:XC6206PxxxMR
- added U103: SRV05-4, Package_TO_SOT_SMD:SOT-23-6, symbol Power_Protection:SRV05-4
Connections:
- new net: J101.A5 (CC1), R101.2
- new net: J101.B5 (CC2), R102.2
- new net: C109.2, J101.S1 (SHIELD), J102.1 (Pin_1), R103.2
- new net: C112.1, Q101.1 (G), R106.2
- new net +3V3: C101.1, C102.1, C103.1, C104.1, C105.1, C106.1, C107.1, C108.1, C111.1, D102.2 (A), R104.1, SW101.1, U101.1 (VBAT), U101.24 (VDD), U101.36 (VDDIO2), U101.48 (VDD), U101.9 (VDDA), U102.2 (VO)
- new net +5V: C110.1, D101.1 (A1), D102.1 (K), F101.1, U102.3 (VI), U103.5 (VP)
- new net BOOT: C112.2, R105.2, SW101.2, U101.44 (BOOT0)
- new net Col_1: U101.31 (PA10)
- new net Col_10: U101.2 (PC13)
- new net Col_11: U101.3 (PC14)
- new net Col_12: U101.4 (PC15)
- new net Col_13: U101.5 (PF0)
- new net Col_2: U101.30 (PA9)
- new net Col_3: U101.29 (PA8)
- new net Col_4: U101.28 (PB15)
- new net Col_5: U101.27 (PB14)
- new net Col_6: U101.25 (PB12)
- new net Col_7: U101.38 (PA15)
- new net Col_8: U101.45 (PB8)
- new net Col_9: U101.46 (PB9)
- new net D+: J101.A6 (D+), J101.B6 (D+), U101.33 (PA12), U103.4 (IO3)
- new net D-: J101.A7 (D-), J101.B7 (D-), U101.32 (PA11), U103.1 (IO1)
- new net GND: C101.2, C102.2, C103.2, C104.2, C105.2, C106.2, C107.2, C108.2, C109.1, C110.2, C111.2, C113.2, D101.2 (A2), J101.A1 (GND), J101.A12 (GND), J101.B1 (GND), J101.B12 (GND), Q101.2 (S), R101.1, R102.1, R103.1, R105.1, R106.1, U101.23 (VSS), U101.35 (VSS), U101.47 (VSS), U101.49 (VSS), U101.8 (VSSA), U102.1 (GND), U103.2 (VN)
- new net NRST: C113.1, Q101.3 (D), R104.2, U101.7 (NRST)
- new net Row_1: U101.39 (PB3)
- new net Row_2: U101.40 (PB4)
- new net Row_3: U101.41 (PB5)
- new net Row_4: U101.42 (PB6)
- new net VBUS: F101.2, J101.A4 (VBUS), J101.A9 (VBUS), J101.B4 (VBUS), J101.B9 (VBUS)
- no-connect marks 0 -> 5

Commit message: working and produced unit
Parts:
- removed U101: STM32F072C8Tx, Package_QFP:LQFP-48_7x7mm_P0.5mm, symbol MCU_ST_STM32F0:STM32F072CBUx
- added U1: STM32F072C8Tx, Package_QFP:LQFP-48_7x7mm_P0.5mm, symbol MCU_ST_STM32F0:STM32F072C8Tx
- renumbered C101 to C1, C110 to C10, C111 to C11, C112 to C12, C113 to C13, C102 to C2, C103 to C3, C104 to C4, C105 to C5, C106 to C6, C107 to C7, C108 to C8, C109 to C9, D101 to D1, D102 to D2, F101 to F1, H101 to H1, H102 to H2, H103 to H3, H104 to H4, H105 to H5, H106 to H6, J101 to J1, J102 to J2, Q101 to Q1, R101 to R1, R102 to R2, R103 to R3, R104 to R4, R105 to R5, R106 to R6, SW101 to SW1, U102 to U2, U103 to U3
Connections:
- net +3V3: now also U1.1 (VBAT), U1.24 (VDD), U1.36 (VDDIO2), U1.48 (VDD), U1.9 (VDDA)
- net BOOT: now also U1.44 (BOOT0)
- net Col_1: now also U1.31 (PA10)
- net Col_10: now also U1.2 (PC13)
- net Col_11: now also U1.3 (PC14)
- net Col_12: now also U1.4 (PC15)
- net Col_13: now also U1.5 (PF0)
- net Col_2: now also U1.30 (PA9)
- net Col_3: now also U1.29 (PA8)
- net Col_4: now also U1.28 (PB15)
- net Col_5: now also U1.27 (PB14)
- net Col_6: now also U1.25 (PB12)
- net Col_7: now also U1.38 (PA15)
- net Col_8: now also U1.45 (PB8)
- net Col_9: now also U1.46 (PB9)
- net D+: now also U1.33 (PA12)
- net D-: now also U1.32 (PA11)
- net GND: now also U1.23 (VSS), U1.35 (VSS), U1.47 (VSS), U1.8 (VSSA)
- net NRST: now also U1.7 (NRST)
- net Row_1: now also U1.39 (PB3)
- net Row_2: now also U1.40 (PB4)
- net Row_3: now also U1.41 (PB5)
- net Row_4: now also U1.42 (PB6)
