File: matrix.sch (KiCad schematic (older format))
At the start: 96 parts, among them K1 KEYSW, K10 KEYSW, K11 KEYSW, K12 KEYSW, K13 KEYSW, K14 KEYSW, K15 KEYSW, K16 KEYSW, K17 KEYSW, K18 KEYSW, K19 KEYSW, K2 KEYSW, K20 KEYSW, K21 KEYSW, K22 KEYSW, K23 KEYSW, K24 KEYSW, K25 KEYSW, K26 KEYSW, K27 KEYSW, K28 KEYSW, K29 KEYSW, K3 KEYSW, K30 KEYSW, K31 KEYSW, K32 KEYSW, K33 KEYSW, K34 KEYSW, K35 KEYSW, K36 KEYSW, K37 KEYSW, K38 KEYSW, K39 KEYSW, K4 KEYSW, K40 KEYSW, K41 KEYSW, K42 KEYSW, K43 KEYSW, K44 KEYSW, K45 KEYSW, K46 KEYSW, K47 KEYSW, K48 KEYSW, K5 KEYSW, K6 KEYSW, K7 KEYSW, K8 KEYSW, K9 KEYSW

Commit message: ready for production
Parts:
- removed D1, D10, D11, D12, D14, D15, D16, D17, D18, D19, D2, D21, D22, D23, D24, D25, D26, D27, D28, D29, D3, D30, D31, D32, D35, D36, D37, D38, D39, D4, D40, D5, D6, D7, D8, D9: D, Diode_SMD:D_0805_2012Metric_Pad1.15x1.40mm_HandSolder, symbol Device:D
- added DD202, DD203, DD204, DD205, DD206, DD207, DD209, DD210, DD211, DD212, DD213, DD214, DD216, DD217, DD218, DD219, DD220, DD221: BAV70, keyboard_parts:SOT23-3_HSOL, symbol Diode:BAV70
- added Stab_1, Stab_2: Stabilizer, Keebio-Parts:2U-StabFlip, symbol Mechanical:MountingHole
- D201: renamed from D13; footprint Diode_SMD:D_0805_2012Metric_Pad1.15x1.40mm_HandSolder -> Diode_SMD:D_SOD-123; JLCPCB (none) -> C8598
- D208: renamed from D20; footprint Diode_SMD:D_0805_2012Metric_Pad1.15x1.40mm_HandSolder -> Diode_SMD:D_SOD-123; JLCPCB (none) -> C8598
- D215: renamed from D33; footprint Diode_SMD:D_0805_2012Metric_Pad1.15x1.40mm_HandSolder -> Diode_SMD:D_SOD-123; JLCPCB (none) -> C8598
- D222: renamed from D34; footprint Diode_SMD:D_0805_2012Metric_Pad1.15x1.40mm_HandSolder -> Diode_SMD:D_SOD-123; JLCPCB (none) -> C8598
- D223: renamed from D41; footprint Diode_SMD:D_0805_2012Metric_Pad1.15x1.40mm_HandSolder -> Diode_SMD:D_SOD-123; JLCPCB (none) -> C8598
- D224: renamed from D42; footprint Diode_SMD:D_0805_2012Metric_Pad1.15x1.40mm_HandSolder -> Diode_SMD:D_SOD-123; JLCPCB (none) -> C8598
- D225: renamed from D43; footprint Diode_SMD:D_0805_2012Metric_Pad1.15x1.40mm_HandSolder -> Diode_SMD:D_SOD-123; JLCPCB (none) -> C8598
- D226: renamed from D44; footprint Diode_SMD:D_0805_2012Metric_Pad1.15x1.40mm_HandSolder -> Diode_SMD:D_SOD-123; JLCPCB (none) -> C8598
- D227: renamed from D45; footprint Diode_SMD:D_0805_2012Metric_Pad1.15x1.40mm_HandSolder -> Diode_SMD:D_SOD-123; JLCPCB (none) -> C8598
- D228: renamed from D46; footprint Diode_SMD:D_0805_2012Metric_Pad1.15x1.40mm_HandSolder -> Diode_SMD:D_SOD-123; JLCPCB (none) -> C8598
- D229: renamed from D47; footprint Diode_SMD:D_0805_2012Metric_Pad1.15x1.40mm_HandSolder -> Diode_SMD:D_SOD-123; JLCPCB (none) -> C8598
- D230: renamed from D48; footprint Diode_SMD:D_0805_2012Metric_Pad1.15x1.40mm_HandSolder -> Diode_SMD:D_SOD-123; JLCPCB (none) -> C8598
- renumbered K1 to K201, K2 to K202, K3 to K203, K4 to K204, K5 to K205, K6 to K206, K7 to K207, K8 to K208, K9 to K209, K10 to K210, K11 to K211, K12 to K212, K13 to K213, K14 to K214, K15 to K215, K16 to K216, K17 to K217, K18 to K218, K19 to K219, K20 to K220, K21 to K221, K22 to K222, K23 to K223, K24 to K224, K25 to K225, K26 to K226, K27 to K227, K28 to K228, K29 to K229, K30 to K230, K31 to K231, K32 to K232, K33 to K233, K35 to K234, K36 to K235, K37 to K236, K38 to K237, K39 to K238, K40 to K239, K34 to K240, K41 to K241, K42 to K242, K43 to K243, K44 to K244, K45 to K245, K46 to K246, K47 to K247, K48 to K248
Connections:
- net Col_1: now reaches K201.1, K214.1, K227.1
- net at K201.2: now also DD202.1 (A)
- net Col_2: now reaches K202.1, K215.1, K228.1
- net Col_2: now also K241.1
- net at K202.2: now also DD202.2 (A)
- net Col_3: now reaches K203.1, K216.1, K229.1
- net Col_3: now also K242.1
- net at K203.2: now also DD203.1 (A)
- net Col_4: now reaches K204.1, K217.1, K230.1
- net Col_4: now also K243.1; no longer K241.1
- net at K204.2: now also DD203.2 (A)
- net Col_5: now reaches K205.1, K218.1, K231.1
- net Col_5: no longer K242.1
- net at K205.2: now also DD204.1 (A)
- net Col_6: now reaches K206.1, K219.1, K232.1
- net Col_6: now also K244.1; no longer K243.1
- net at K206.2: now also DD204.2 (A)
- net Col_7: now reaches K207.1, K240.1
- net Col_7: now also K220.1, K233.1; no longer K245.1
- net at K207.2: now also D201.2 (A)
- net Col_8: now reaches K208.1, K221.1, K234.1
- net Col_8: now also K245.1; no longer K246.1
- net at K208.2: now also DD205.1 (A)
- net Col_9: now reaches K209.1, K222.1, K235.1
- net Col_9: no longer K247.1
- net at K209.2: now also DD205.2 (A)
- net Col_10: now reaches K210.1, K223.1, K236.1
- net Col_10: now also K246.1; no longer K248.1
- net at K210.2: now also DD206.1 (A)
- net Col_11: now reaches K211.1, K224.1, K237.1
- net Col_11: now also K247.1
- net at K211.2: now also DD206.2 (A)
- net Col_12: now reaches K212.1, K225.1, K238.1
- net Col_12: now also K248.1
- net at K212.2: now also DD207.1 (A)
- net Col_13: now reaches K213.1, K226.1, K239.1
- net at K213.2: now also DD207.2 (A); no longer D201.2 (A)
- net at K214.2: now also DD209.1 (A)
- net at K215.2: now also DD209.2 (A)
- net at K216.2: now also DD210.1 (A)
- net at K217.2: now also DD210.2 (A)
- net at K218.2: now also DD211.1 (A)
- net at K219.2: now also DD211.2 (A)
- net at K221.2: now also DD212.1 (A)
- net at K222.2: now also DD212.2 (A)
- net at K223.2: now also DD213.1 (A)
- net at K224.2: now also DD213.2 (A)
- net at K225.2: now also DD214.1 (A)
- net at K226.2: now also DD214.2 (A)
- net at K227.2: now also DD216.2 (A)
- net at K228.2: now also DD216.1 (A)
- net at K229.2: now also DD217.2 (A)
- net at K230.2: now also DD217.1 (A)
- net at K231.2: now also DD218.2 (A)
- net at K232.2: now also DD218.1 (A)
- net at K234.2: now also DD219.2 (A)
- net at K235.2: now also DD219.1 (A)
- net at K236.2: now also DD220.2 (A)
- net at K237.2: now also DD220.1 (A)
- net at K238.2: now also DD221.2 (A)
- net at K239.2: now also DD221.1 (A)
- net Row_1: now reaches D201.1 (K)
- net Row_1: now also DD202.3 (K), DD203.3 (K), DD204.3 (K), DD205.3 (K), DD206.3 (K), DD207.3 (K)
- net Row_2: now reaches D208.1 (K)
- net Row_2: now also DD209.3 (K), DD210.3 (K), DD211.3 (K), DD212.3 (K), DD213.3 (K), DD214.3 (K)
- net Row_3: now reaches D215.1 (K)
- net Row_3: now also DD216.3 (K), DD217.3 (K), DD218.3 (K), DD219.3 (K), DD220.3 (K), DD221.3 (K); no longer D222.1 (K)
- net Row_4: now reaches D223.1 (K), D224.1 (K), D225.1 (K), D226.1 (K), D227.1 (K), D228.1 (K), D229.1 (K), D230.1 (K)
- net Row_4: now also D222.1 (K)
Other:
- moved on the sheet: D201, D208, D215, D222, D223, D224, D225, D226, D227, D228, D229, D230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

Commit message: working and produced unit
Parts:
- renumbered D226 to D10, D227 to D11, D228 to D12, D229 to D13, D230 to D14, D201 to D3, D208 to D4, D215 to D5, D222 to D6, D223 to D7, D224 to D8, D225 to D9, DD202 to DD1, DD212 to DD10, DD213 to DD11, DD214 to DD12, DD216 to DD13, DD217 to DD14, DD218 to DD15, DD219 to DD16, DD220 to DD17, DD221 to DD18, DD203 to DD2, DD204 to DD3, DD205 to DD4, DD206 to DD5, DD207 to DD6, DD209 to DD7, DD210 to DD8, DD211 to DD9, K201 to K1, K210 to K10, K211 to K11, K212 to K12, K213 to K13, K214 to K14, K215 to K15, K216 to K16, K217 to K17, K218 to K18, K219 to K19, K202 to K2, K220 to K20, K221 to K21, K222 to K22, K223 to K23, K224 to K24, K225 to K25, K226 to K26, K227 to K27, K228 to K28, K229 to K29, K203 to K3, K230 to K30, K231 to K31, K232 to K32, K233 to K33, K234 to K34, K235 to K35, K236 to K36, K237 to K37, K238 to K38, K239 to K39, K204 to K4, K240 to K40, K241 to K41, K242 to K42, K243 to K43, K244 to K44, K245 to K45, K246 to K46, K247 to K47, K248 to K48, K205 to K5, K206 to K6, K207 to K7, K208 to K8, K209 to K9
